File: GAHT greenhouse controls.kicad_sch (KiCad schematic)
At the start: 7 parts, among them U2 DS18B20, U3 DS18B20, U4 DS18B20, U5 ESP32-S3-WROOM-1

Commit message: Add files via upload
Connections:
- net +3.3V: now also U1.6 (3.3V)
- net GND: no longer U1.8 (GND)
- net at U1.2 (MISO): now also U5.21 (IO13); no longer U5.13 (IO19)
- net at U1.3 (SCK): now also U5.20 (IO12); no longer U5.12 (IO8)
- net at U1.4 (MOSI): now also U5.19 (IO11); no longer U5.11 (IO18)
- net at U1.5 (CS): now also U5.18 (IO10); no longer U5.10 (IO17)
Other:
- moved on the sheet: C1, R1, U1, U2, U3, U4
